File: robomow_usb.sch (EAGLE design)
At the start: 31 parts, among them IC1 FT231XS-R, J1 RJ11-2L-B, U1 SN65HVD1176

Commit message: Fixup input filtering
Parts:
- J1: value RJ11-2L-B -> RJ11NO_DIMENSION; device con-tycoelectronics:RJ11-2L-B -> con-tycoelectronics:RJ11NO_DIMENSION
- PWR, RX, TX: value (none) -> LED_0603
Connections:
- new net VUSB_CONN: C6.1, CR3.2, JUSB.VBUS, R2.1
- net VUSB: no longer C6.1, CR3.2, JUSB.VBUS, R2.1
Other:
- note added: "RS-485 R+"
- note added: "RS-485 R-"
- note added: "RS-485 T+"
- note added: "RS-485 T-"
- note added: "Sorensen DLM series RS-485 pinout"
- moved on the sheet: PWR, R10, R11, R12, R13, R14, R15, R4, R8, RX, TX
